File: boss_ce2/boss_ce2_assembly/boss_ce2_assembly/boss_ce2_assembly.kicad_pcb (KiCad board)
At the start: 2 copper layers, 75 x 100 mm, 111 parts, among them J1 INPUT, J2 OUTPUT, Q1 BC239/BC238, Q2 BC239/BC238, Q3 BC239/BC238, Q4 2SC945, Q5 2SC945, Q6 2SC945, Q7 2SC945, Q8 2SC945, Q9 2SK30A, SW1 FOOTSWITCH, U1 JRC4558D, U2 MN3007, U3 MN3101, U4 TL022CP, U5 TL022CP

Commit message: push test
Connections:
- C11 pad 2: GND -> +9VA
- C13 pad 2: GND -> +9VA
- C18 pad 2: GND -> +9VA
- C21 pad 2: GND -> +9VA
- C23 pad 2: GND -> +9VA
- C28 pad 1: GND -> +9VA
- C29 pad 2: GND -> +9VA
- C30 pad 2: GND -> +9VA
- C6 pad 1: GND -> +9VA
- C8 pad 1: GND -> +9VA
- C9 pad 2: GND -> +9VA
- D3 pad 1: GND -> +9VA
- D7 pad 2: GND -> +9VA
- J1 pad S: GND -> +9VA
- J2 pad S: GND -> +9VA
- Q5 pad 3: GND -> +9VA
- Q8 pad 3: GND -> +9VA
- R12 pad 1: GND -> +9VA
- R19 pad 1: GND -> +9VA
- R26 pad 2: GND -> +9VA
- R28 pad 2: GND -> +9VA
- R3 pad 2: GND -> +9VA
- R37 pad 1: GND -> +9VA
- R47 pad 2: GND -> +9VA
- R48 pad 2: GND -> +9VA
- SW1 pad 1: GND -> +9VA
- U1 pad 4: GND -> +9VA
- U2 pad 5: GND -> +9VA
- U3 pad 3: GND -> +9VA
- U4 pad 4: GND -> +9VA
- U5 pad 4: GND -> +9VA
Routing:
- net +9VA: track 134.4 -> 439.1 mm, vias 6 -> 0
- net +9V: track 49.4 -> 234.8 mm, vias 2 -> 1
- net +4V: track 13.4 -> 179.6 mm
- net Net-(R32-Pad2): track 72.3 -> 90.3 mm
- net Net-(C16-Pad2): track 80.7 -> 94.0 mm, vias 2 -> 0
- net Net-(U4-1OUT): track 69.9 -> 80.4 mm, vias 1 -> 0
- net Net-(U5-1IN+): track 26.8 -> 36.5 mm
- net Net-(R35-Pad2): track 56.8 -> 49.1 mm, vias 3 -> 1
- net GND: track 6.50 -> 0.00 mm
- net Net-(CONN1-Pad1): track 65.3 -> 59.6 mm, vias 1 -> 0
- net Net-(C15-Pad1): track 79.2 -> 74.9 mm, vias 4 -> 0
- net Net-(U2-IN): track 4.36 -> 8.62 mm
- net Net-(C17-Pad1): track 73.1 -> 77.3 mm, vias 1 -> 0
- net Net-(C24-Pad2): track 15.5 -> 19.6 mm, vias 1 -> 0
- net Net-(Q2-E): track 18.0 -> 21.9 mm
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